File: atmega embedded main 2.brd (EAGLE design)
At the start: 313.5 x 125.9 mm, 146 parts, among them IC1 ATMEGA328PROUND, K1 SWITCH, K100 SWITCH, K101 SWITCH, K102 SWITCH, K103 SWITCH, K104 SWITCH, K105 SWITCH, K106 SWITCH, K107 SWITCH, K108 SWITCH, K109 SWITCH, K110 SWITCH, K111 SWITCH, K112 SWITCH, K113 SWITCH, K114 SWITCH, K115 SWITCH, K116 SWITCH, K117 SWITCH, K118 SWITCH, K119 SWITCH, K120 SWITCH, K121 SWITCH, K122 SWITCH, K123 SWITCH, K125 SWITCH, K126 SWITCH, K127 SWITCH, K128 SWITCH, K129 SWITCH, K130 SWITCH, K2 SWITCH, K3 SWITCH, K60 SWITCH, K67 SWITCH, K68 SWITCH, K69 SWITCH, K70 SWITCH, K71 SWITCH, K72 SWITCH, K73 SWITCH, K74 SWITCH, K75 SWITCH, K76 SWITCH, K77 SWITCH, K78 SWITCH, K79 SWITCH, K80 SWITCH, K81 SWITCH, K82 SWITCH, K83 SWITCH, K84 SWITCH, K85 SWITCH, K86 SWITCH, K87 SWITCH, K88 SWITCH, K89 SWITCH, K90 SWITCH, K91 SWITCH, K92 SWITCH, K93 SWITCH, K94 SWITCH, K95 SWITCH, K96 SWITCH, K98 SWITCH, K99 SWITCH

Commit message: Fixed errors and made adjustments for USB
Parts:
- removed D3: (no value), adafruit:SMADIODE
- removed K1, K2, K3: SWITCH, keyboard_switch:KAILH_LOW_PROFILE
- added D111, D86: (no value), adafruit:SMADIODE
- added K124, K97: SWITCH, keyboard_switch:KAILH_LOW_PROFILE
- added R1: 1M, eagle-ltspice:R1206
- added R2: 1.5K, eagle-ltspice:R1206
- D1, D2: value (none) -> 3.6; device adafruit:SMADIODE -> diode:SMB
- R6, R7: value 22 -> 68; device adafruit:M0805 -> eagle-ltspice:R1206
- moved D2 231.3 mm to (61.8, 111.6), flipped to the top, turned to 90 degrees
- moved D1 207.2 mm to (71.2, 111.6), flipped to the top, turned to 90 degrees
- moved C3 23.9 mm to (130.6, 104.5)
- moved C4 23.9 mm to (125.9, 104.5)
- moved C5 23.9 mm to (121.1, 104.5)
- moved C6 23.9 mm to (116.4, 104.5)
- moved C7 23.9 mm to (111.6, 104.5)
- moved R5 23.8 mm to (102.1, 104.5)
- moved S1 23.8 mm to (106.9, 97.4)
- moved U1 21.4 mm to (95.0, 115.2)
- moved D129 19.0 mm to (173.4, 4.75)
- moved D130 19.0 mm to (106.9, 4.75)
- moved K129 19.0 mm to (180.5, 0.00)
- moved K130 19.0 mm to (114.0, 0.00)
- moved D87 9.57 mm to (30.9, 23.8)
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Connections:
- removed net N$69: D1.C, K1.P$1
- net COL10: no longer K1.P$2
- net COL2: no longer K3.P$2
- net COL4: now also K97.P$2
- net COL6: no longer K128.P$2
- net COL7: now also K124.P$2, K128.P$2; no longer K123.P$2
- net COL8: now also K123.P$2; no longer K117.P$2
- net COL9: now also K117.P$2; no longer K2.P$2
- net D+: now also D1.C, R1.1
- net D-: now also D2.C, R2.2
- net GND: now also D1.A, D2.A, R1.2
- net N$23: now also D86.C, K97.P$1; no longer D3.C, K3.P$1
- net N$47: now also D111.C, K124.P$1; no longer D2.C, K2.P$1
- net ROW4: now also IC1.16; no longer D1.A, D3.A, IC1.17
- net ROW5: now also D111.A, D86.A
- net ROW6: now also IC1.17; no longer D2.A, IC1.16
- net VCC: now also R2.1
Routing:
- net ROW5: track 629.5 -> 771.5 mm
- net COL6: track 387.7 -> 277.7 mm
- net ROW6: track 401.7 -> 477.0 mm
- net ROW3: track 601.5 -> 646.0 mm
- net GND: track 148.2 -> 185.5 mm
- net ROW4: track 625.0 -> 658.2 mm
- net COL7: track 359.5 -> 386.5 mm
- net D+: track 39.7 -> 65.6 mm
- net VCC: track 114.8 -> 139.8 mm
- net ROW2: track 576.4 -> 600.6 mm
- net N$15: track 36.2 -> 60.0 mm
- net D-: track 46.8 -> 68.9 mm
- net ROW7: track 279.1 -> 260.1 mm
- net COL4: track 301.2 -> 319.3 mm
- net COL9: track 443.4 -> 428.9 mm
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