File: atmega embedded main - za drugog Marka.brd (EAGLE design)
At the start: 313.5 x 125.9 mm, 150 parts, among them IC1 ATMEGA328PROUND, K100 SWITCH, K101 SWITCH, K102 SWITCH, K103 SWITCH, K104 SWITCH, K105 SWITCH, K106 SWITCH, K107 SWITCH, K108 SWITCH, K109 SWITCH, K110 SWITCH, K111 SWITCH, K112 SWITCH, K113 SWITCH, K114 SWITCH, K115 SWITCH, K116 SWITCH, K117 SWITCH, K118 SWITCH, K119 SWITCH, K120 SWITCH, K121 SWITCH, K122 SWITCH, K123 SWITCH, K124 SWITCH, K125 SWITCH, K126 SWITCH, K127 SWITCH, K128 SWITCH, K129 SWITCH, K130 SWITCH, K60 SWITCH, K67 SWITCH, K68 SWITCH, K69 SWITCH, K70 SWITCH, K71 SWITCH, K72 SWITCH, K73 SWITCH, K74 SWITCH, K75 SWITCH, K76 SWITCH, K77 SWITCH, K78 SWITCH, K79 SWITCH, K80 SWITCH, K81 SWITCH, K82 SWITCH, K83 SWITCH, K84 SWITCH, K85 SWITCH, K86 SWITCH, K87 SWITCH, K88 SWITCH, K89 SWITCH, K90 SWITCH, K91 SWITCH, K92 SWITCH, K93 SWITCH, K94 SWITCH, K95 SWITCH, K96 SWITCH, K97 SWITCH, K98 SWITCH, K99 SWITCH

Commit message: Finalized logic and started work on Marko's layout
Parts:
- removed D129, D130: (no value), adafruit:SMADIODE
- removed K129, K130: SWITCH, keyboard_switch:KAILH_LOW_PROFILE
- added D3, D4, D5: (no value), adafruit:SMADIODE
- added K1, K2, K3: SWITCH, keyboard_switch:KAILH_LOW_PROFILE
- moved D87 9.57 mm to (22.6, 28.5)
- moved D111 9.50 mm to (192.4, 4.75)
- moved D125 9.50 mm to (239.9, 23.8)
- moved D128 9.50 mm to (288.6, 47.5)
- moved D86 9.50 mm to (87.9, 4.75)
- moved D97 9.50 mm to (129.4, 19.0)
- moved D98 9.50 mm to (165.1, 19.0)
- moved K117 9.50 mm to (294.5, 38.0)
- moved K118 9.50 mm to (171.0, 9.50)
- moved K122 9.50 mm to (247.0, 19.0)
- moved K124 9.50 mm to (199.5, 0.00)
- moved K60 9.50 mm to (9.50, 76.0)
- moved K73 9.50 mm to (9.50, 57.0)
- moved K80 9.50 mm to (9.50, 38.0)
- moved K87 9.50 mm to (9.50, 19.0)
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Connections:
- new net N$71: D3.C, K1.P$1
- net COL10: now also K3.P$2
- net COL2: now also K1.P$2
- net COL5: no longer K130.P$2
- net COL6: now also K128.P$2; no longer K129.P$2
- net COL7: now also K123.P$2; no longer K128.P$2
- net COL8: now also K117.P$2; no longer K123.P$2
- net COL9: now also K2.P$2; no longer K117.P$2
- net N$26: now also D5.C, K3.P$1; no longer D129.C, K129.P$1
- net N$35: now also D4.C, K2.P$1; no longer D130.C, K130.P$1
- net ROW4: now also D3.A, D5.A, IC1.15; no longer IC1.16
- net ROW5: now also IC1.17; no longer D129.A, D130.A, IC1.15
- net ROW6: now also D4.A, IC1.16; no longer IC1.17
Routing:
- net ROW5: track 766.2 -> 553.4 mm
- net COL6: track 277.7 -> 397.5 mm
- net ROW4: track 658.2 -> 774.0 mm
- net COL5: track 319.6 -> 276.8 mm, vias 1 -> 2
- net ROW7: track 260.1 -> 279.1 mm
- net COL1: track 203.5 -> 191.8 mm
- net COL2: track 316.2 -> 307.4 mm
- net N$71: track 0.00 -> 5.29 mm
- net ROW6: track 477.0 -> 472.1 mm
- net COL9: track 431.2 -> 426.9 mm
- net COL4: track 323.2 -> 320.0 mm
- net COL3: track 314.8 -> 311.8 mm
- net ROW1: track 382.2 -> 379.6 mm
- net N$6: track 3.76 -> 5.52 mm
- net COL7: track 389.5 -> 390.5 mm
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Other:
- board size 313.5 x 125.9 mm -> 311.1 x 125.9 mm

Commit message: Finished Marko's board and fixed some errors.
Parts:
- moved K104 9.50 mm to (285.0, 76.0)
- moved K117 9.50 mm to (285.0, 38.0)
- moved K123 9.50 mm to (285.0, 19.0)
- moved K128 9.50 mm to (285.0, 0.00)
- moved K2 9.50 mm to (285.0, 57.0)
- moved D104 2.38 mm to (290.9, 9.50), turned to 180 degrees
- moved D115 2.38 mm to (290.9, 85.5), turned to 180 degrees
- moved D127 2.38 mm to (290.9, 28.5), turned to 180 degrees
- moved D128 2.38 mm to (290.9, 47.5), turned to 180 degrees
- moved D4 2.38 mm to (290.9, 66.5), turned to 180 degrees
Routing:
- net ROW5: track 553.4 -> 809.7 mm
- net ROW4: track 774.0 -> 833.8 mm
- net ROW3: track 647.0 -> 676.0 mm
- net ROW2: track 600.6 -> 629.4 mm
- net COL6: track 397.5 -> 387.2 mm
- net COL10: track 340.8 -> 330.8 mm
- net COL8: track 404.9 -> 395.5 mm
- net COL7: track 390.5 -> 381.2 mm
- net COL9: track 426.9 -> 417.8 mm
- net ROW6: track 472.1 -> 479.6 mm

Commit message: Wired up connectors
Parts:
- moved C6 10.1 mm to (112.8, 113.4)
- moved C7 10.1 mm to (109.2, 113.4)
- moved S1 7.45 mm to (102.0, 108.7), turned to 180 degrees
- moved C5 7.44 mm to (116.4, 113.4), turned to 270 degrees
- moved D116 5.46 mm to (165.1, 80.0)
- moved R2 5.46 mm to (91.9, 104.5)
- moved R5 5.46 mm to (96.7, 104.5)
- moved U1 5.46 mm to (89.5, 115.2)
- moved C3 3.61 mm to (123.5, 113.4), turned to 270 degrees
- moved C4 2.97 mm to (119.9, 113.4), turned to 270 degrees
- moved D72 1.78 mm to (129.4, 83.7)
Connections:
- net N$15 renamed RESET
Routing:
- net VCC: track 146.4 -> 67.4 mm
- net GND: track 273.2 -> 205.4 mm
- net ROW2: track 629.4 -> 565.8 mm
- net ROW3: track 676.0 -> 617.1 mm
- net ROW6: track 479.6 -> 447.1 mm
- net ROW5: track 809.7 -> 779.7 mm
- net ROW1: track 379.6 -> 349.8 mm
- net COL8: track 395.5 -> 367.5 mm
- net ROW4: track 833.8 -> 806.4 mm
- net COL7: track 381.2 -> 354.4 mm
- net COL6: track 387.2 -> 360.6 mm
- net RESET: track 67.8 -> 93.8 mm
- net COL10: track 330.8 -> 309.4 mm
- net COL9: track 417.8 -> 397.1 mm, vias 3 -> 2
- net D-: track 68.9 -> 63.4 mm
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
Commit message: Rewired some stuff
Parts:
- moved D99 6.42 mm to (186.4, 86.1)
- moved D72 1.19 mm to (130.6, 83.7)
Routing:
- net COL9: track 397.1 -> 479.6 mm
- net COL2: track 305.6 -> 387.8 mm
- net COL8: track 367.5 -> 440.4 mm
- net COL3: track 311.8 -> 371.8 mm
- net COL7: track 354.4 -> 408.0 mm, vias 3 -> 2
- net COL4: track 320.0 -> 365.8 mm, vias 2 -> 1
- net GND: track 205.4 -> 210.4 mm, vias 2 -> 1
- net D-: track 63.4 -> 60.6 mm
- net COL10: track 309.4 -> 306.6 mm, vias 2 -> 1
- net ROW4: track 806.4 -> 803.6 mm
- net ROW1: track 349.8 -> 352.3 mm
- net ROW7: track 277.7 -> 276.3 mm
- net ROW2: track 565.8 -> 564.4 mm
- net N$36: track 3.99 -> 5.08 mm
- net COL6: track 360.6 -> 359.7 mm
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