File: atmega embedded main - za drugog Marka.brd (EAGLE design)
At the start: 311.1 x 125.9 mm, 152 parts, among them IC1 ATMEGA328PROUND, K1 SWITCH, K100 SWITCH, K101 SWITCH, K102 SWITCH, K103 SWITCH, K104 SWITCH, K105 SWITCH, K106 SWITCH, K107 SWITCH, K108 SWITCH, K109 SWITCH, K110 SWITCH, K111 SWITCH, K112 SWITCH, K113 SWITCH, K114 SWITCH, K115 SWITCH, K116 SWITCH, K117 SWITCH, K118 SWITCH, K119 SWITCH, K120 SWITCH, K121 SWITCH, K122 SWITCH, K123 SWITCH, K124 SWITCH, K125 SWITCH, K126 SWITCH, K127 SWITCH, K128 SWITCH, K2 SWITCH, K3 SWITCH, K60 SWITCH, K67 SWITCH, K68 SWITCH, K69 SWITCH, K70 SWITCH, K71 SWITCH, K72 SWITCH, K73 SWITCH, K74 SWITCH, K75 SWITCH, K76 SWITCH, K77 SWITCH, K78 SWITCH, K79 SWITCH, K80 SWITCH, K81 SWITCH, K82 SWITCH, K83 SWITCH, K84 SWITCH, K85 SWITCH, K86 SWITCH, K87 SWITCH, K88 SWITCH, K89 SWITCH, K90 SWITCH, K91 SWITCH, K92 SWITCH, K93 SWITCH, K94 SWITCH, K95 SWITCH, K96 SWITCH, K97 SWITCH, K98 SWITCH, K99 SWITCH

Commit message: Test 1
Parts:
- moved D87 23.8 mm to (21.4, 4.75)
- moved D84 19.0 mm to (59.4, 4.75)
- moved D85 19.0 mm to (78.4, 4.75)
- moved D86 19.0 mm to (106.9, 4.75)
- moved K88 19.0 mm to (28.5, 0.00)
- moved K94 19.0 mm to (47.5, 0.00)
- moved K95 19.0 mm to (66.5, 0.00)
- moved K96 19.0 mm to (85.5, 0.00)
- moved K97 19.0 mm to (114.0, 0.00)
- moved D82 18.8 mm to (3.56, 28.2)
- moved D83 18.4 mm to (40.4, 4.75)
- moved D81 11.0 mm to (9.00, 18.9), turned to 270 degrees
- moved K87 9.75 mm to (19.2, 19.0)
- moved D97 9.50 mm to (129.4, 28.5)
- moved K92 9.50 mm to (123.5, 19.0)
Connections:
- net COL1: now also K87.P$2; no longer K94.P$2
- net COL2: now also K94.P$2; no longer K95.P$2
- net COL3: now also K95.P$2; no longer K96.P$2
- net COL4: now also K96.P$2; no longer K87.P$2, K97.P$2
- net ROW4: now also D81.A; no longer D87.A
- net ROW5: now also D87.A; no longer D86.A
- net ROW6: no longer D81.A
- net ROW7: now also D86.A
Routing:
- net COL4: track 365.8 -> 191.6 mm
- net ROW5: track 779.7 -> 659.4 mm
- net COL5: track 276.8 -> 185.9 mm, vias 2 -> 1
- net ROW4: track 803.6 -> 737.7 mm
- net COL1: track 191.8 -> 152.7 mm
- net COL3: track 371.8 -> 351.9 mm
- net ROW6: track 447.1 -> 427.3 mm
- net COL2: track 387.8 -> 368.3 mm
- net ROW7: track 276.3 -> 266.8 mm
- net N$4: track 5.16 -> 11.8 mm
- net N$5: track 5.16 -> 0.18 mm

Commit message: Test2
Parts:
- moved K3 26.0 mm to (284.8, 1.00)
- moved D5 23.4 mm to (276.4, 8.19)
- moved D104 23.4 mm to (268.1, 14.5)
- moved D82 23.3 mm to (2.06, 5.00)
- moved D119 19.1 mm to (199.6, 14.5), turned to 180 degrees
- moved K124 19.0 mm to (180.5, 0.75)
- moved D111 18.8 mm to (173.6, 5.50)
- moved D112 18.8 mm to (202.1, 5.50)
- moved D113 18.8 mm to (221.1, 5.50)
- moved D114 18.8 mm to (240.1, 5.50)
- moved K125 18.8 mm to (209.2, 0.75)
- moved K126 18.8 mm to (228.2, 0.75)
- moved K127 18.8 mm to (247.2, 0.75)
- moved K128 18.8 mm to (266.2, 0.75)
- moved D81 10.4 mm to (3.50, 27.8), turned to 0 degrees
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Connections:
- removed net N$66: D127.C, K123.P$1
- new net N$15: D98.C, K118.P$2
- net COL1: now also D86.A
- net COL2: now also K72.P$1; no longer K72.P$2
- net COL6: now also K118.P$1, K119.P$1; no longer K118.P$2, K119.P$2
- net COL7: now also K123.P$1; no longer K123.P$2
- net N$36: now also K72.P$2; no longer K72.P$1
- net N$41: now also D119.C, K119.P$2; no longer D98.C, K118.P$1
- net N$43: now also D127.C, K123.P$2; no longer D119.C, K119.P$1
- net ROW4: now also D82.A; no longer D81.A
- net ROW6: now also D81.A; no longer D82.A
- net ROW7: now also K97.P$2; no longer D86.A
Routing:
- net COL3: track 351.9 -> 52.2 mm, vias 2 -> 0
- net COL5: track 185.9 -> 5.52 mm, vias 1 -> 0
- net COL2: track 368.3 -> 190.5 mm, vias 2 -> 1
- net COL4: track 191.6 -> 32.7 mm, vias 1 -> 0
- net ROW5: track 659.4 -> 816.4 mm, vias 2 -> 3
- net COL7: track 408.0 -> 313.3 mm
- net COL9: track 479.6 -> 385.5 mm
- net COL8: track 440.4 -> 360.0 mm
- net COL6: track 359.7 -> 294.7 mm
- net COL1: track 152.7 -> 93.2 mm
- net ROW3: track 617.1 -> 673.7 mm, vias 2 -> 1
- net ROW2: track 564.4 -> 615.0 mm, vias 2 -> 1
- net ROW6: track 427.3 -> 474.1 mm, vias 2 -> 1
- net COL10: track 306.6 -> 266.6 mm
- net ROW1: track 352.3 -> 319.9 mm
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
Commit message: Horrible design
Parts:
- moved D127 21.2 mm to (270.0, 24.9), turned to 90 degrees
- moved D119 18.8 mm to (184.0, 25.0), turned to 90 degrees
- moved D91 15.8 mm to (75.1, 44.1), turned to 90 degrees
- moved D72 13.1 mm to (118.4, 81.2), turned to 45 degrees
- moved D115 12.7 mm to (279.1, 81.0), turned to 0 degrees
- moved D89 12.6 mm to (52.2, 47.1), turned to 180 degrees
- moved D97 12.4 mm to (117.5, 25.0), turned to 90 degrees
- moved D128 12.1 mm to (279.5, 43.5), turned to 90 degrees
- moved D4 12.1 mm to (279.6, 62.5), turned to 0 degrees
- moved D96 12.0 mm to (118.0, 44.0), turned to 90 degrees
- moved D104 11.1 mm to (260.5, 6.50), turned to 90 degrees
- moved D73 10.9 mm to (118.5, 66.0), turned to 90 degrees
- moved D83 10.7 mm to (50.0, 9.50), turned to 180 degrees
- moved D81 10.1 mm to (12.7, 23.6)
- moved D88 7.10 mm to (26.0, 48.0)
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Connections:
- net COL2: now also K82.P$1; no longer K82.P$2
- net COL3: now also K83.P$1; no longer K83.P$2
- net COL6: now also K118.P$2; no longer K118.P$1
- net N$11: now also K82.P$2; no longer K82.P$1
- net N$15: now also K118.P$1; no longer K118.P$2
- net N$22: now also K83.P$2; no longer K83.P$1
Routing:
- net COL3: track 52.2 -> 541.4 mm, vias 0 -> 10
- net COL5: track 5.52 -> 402.2 mm, vias 0 -> 4
- net COL4: track 32.7 -> 419.7 mm, vias 0 -> 5
- net COL1: track 93.2 -> 387.5 mm, vias 1 -> 5
- net ROW2: track 615.0 -> 369.2 mm, vias 1 -> 8
- net COL2: track 190.5 -> 433.6 mm, vias 1 -> 10
- net COL6: track 294.7 -> 523.4 mm, vias 2 -> 3
- net ROW4: track 757.3 -> 574.3 mm, vias 3 -> 6
- net VCC: track 61.8 -> 218.8 mm, vias 1 -> 2
- net COL7: track 313.3 -> 456.9 mm, vias 2 -> 6
- net COL8: track 360.0 -> 501.9 mm, vias 3 -> 5
- net ROW3: track 673.7 -> 533.7 mm, vias 1 -> 4
- net COL9: track 385.5 -> 524.4 mm, vias 2 -> 7
- net ROW6: track 474.1 -> 590.7 mm, vias 1 -> 9
- net COL10: track 266.6 -> 382.4 mm, vias 1 -> 5
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
Commit message: Less horrible
Routing:
- net COL2: track 433.6 -> 442.7 mm
- net COL5: track 402.2 -> 405.1 mm
- net COL1: track 387.5 -> 390.3 mm
- net ROW4: track 574.3 -> 576.2 mm
- net COL3: track 541.4 -> 542.4 mm
Changed lines of the file:
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@@
 <wire x1="105.6505" y1="6.5" x2="104.4505" y2="5.3" width="2" layer="16"/>
 <wire x1="104.4505" y1="5.3" x2="104.4505" y2="-7.15" width="2" layer="16"/>
-<wire x1="45.15" y1="-7.15" x2="104.4505" y2="-7.15" width="2" layer="16"/>
-<wire x1="34.3" y1="3.7" x2="38" y2="0" width="2" layer="16"/>
-<wire x1="38" y1="0" x2="45.15" y2="-7.15" width="2" layer="16"/>
-<wire x1="33.8" y1="3.7" x2="34.3" y2="3.7" width="2" layer="16"/>
+<wire x1="41.26" y1="-7.15" x2="104.4505" y2="-7.15" width="2" layer="16"/>
+<wire x1="36.16" y1="3.7" x2="38" y2="1.86" width="2" layer="16"/>
+<wire x1="38" y1="-3.89" x2="38.1" y2="-3.99" width="2" layer="16"/>
+<wire x1="38.1" y1="-3.99" x2="41.26" y2="-7.15" width="2" layer="16"/>
+<wire x1="33.8" y1="3.7" x2="36.16" y2="3.7" width="2" layer="16"/>
 <wire x1="33.8" y1="3.7" x2="33.75" y2="3.75" width="2" layer="16"/>
 <wire x1="15.04" y1="88.7" x2="15.04" y2="97.17" width="2" layer="16"/>
@@
 <wire x1="22.8" y1="42.6" x2="19" y2="46.4" width="2" layer="16"/>
 <wire x1="22.8" y1="42.6" x2="22.7" y2="41.7" width="2" layer="16"/>
-<wire x1="34.3" y1="-3.7" x2="38" y2="0" width="2" layer="16"/>
-<wire x1="3.7" y1="-3.7" x2="34.3" y2="-3.7" width="2" layer="16"/>
+<wire x1="37.19" y1="-4.9" x2="38.1" y2="-3.99" width="2" layer="16"/>
+<wire x1="4.9" y1="-4.9" x2="37.19" y2="-4.9" width="2" layer="16"/>
 <via x="11.52" y="103.97" extent="1-16" drill="2"/>
 <via x="9.1" y="88.7" extent="1-16" drill="2"/>
@@
 <wire x1="19.11" y1="38.01" x2="18.56" y2="37.46" width="2" layer="16"/>
 <wire x1="18.56" y1="37.46" x2="15.1" y2="34" width="2" layer="16"/>
-<wire x1="0" y1="0" x2="3.7" y2="-3.7" width="2" layer="16"/>
+<wire x1="0" y1="0" x2="4.9" y2="-4.9" width="2" layer="16"/>
 <wire x1="15.04" y1="97.17" x2="11.52" y2="100.69" width="2" layer="16"/>
 <wire x1="11.52" y1="103.97" x2="11.52" y2="100.69" width="2" layer="16"/>
+<wire x1="38" y1="-3.89" x2="38" y2="1.86" width="2" layer="16"/>
 </signal>
 <signal name="COL2">
@@
 <contactref element="K94" pad="P$2"/>
 <contactref element="K72" pad="P$1"/>
-<wire x1="46.6" y1="3.7" x2="52.7" y2="3.7" width="2" layer="16"/>
-<wire x1="45.1" y1="5.2" x2="46.6" y2="3.7" width="2" layer="16"/>
-<wire x1="45.1" y1="11.2" x2="45.1" y2="5.2" width="2" layer="16"/>
-<wire x1="50" y1="16.1" x2="45.1" y2="11.2" width="2" layer="16"/>
-<wire x1="54.1" y1="16.1" x2="50" y2="16.1" width="2" layer="16"/>
-<wire x1="55.9" y1="17.9" x2="54.1" y2="16.1" width="2" layer="16"/>
-<wire x1="55.9" y1="20.1" x2="55.9" y2="17.9" width="2" layer="16"/>
-<wire x1="53.3" y1="22.7" x2="55.9" y2="20.1" width="2" layer="16"/>
-<wire x1="52.8" y1="22.7" x2="53.3" y2="22.7" width="2" layer="16"/>
+<wire x1="42.63" y1="3.7" x2="52.7" y2="3.7" width="2" layer="16"/>
+<wire x1="42.63" y1="13.67" x2="42.63" y2="3.7" width="2" layer="16"/>
+<wire x1="43.58" y1="13.68" x2="43.1" y2="13.2" width="2" layer="16"/>
+<wire x1="56.87" y1="13.68" x2="43.58" y2="13.68" width="2" layer="16"/>
+<wire x1="56.87" y1="21.08" x2="56.87" y2="13.68" width="2" layer="16"/>
+<wire x1="55.25" y1="22.7" x2="56.87" y2="21.08" width="2" layer="16"/>
+<wire x1="52.8" y1="22.7" x2="55.25" y2="22.7" width="2" layer="16"/>
 <wire x1="52.7" y1="3.7" x2="52.75" y2="3.75" width="2" layer="16"/>
 <wire x1="52.8" y1="22.7" x2="52.75" y2="22.75" width="2" layer="16"/>
@@
 <wire x1="57" y1="84.09" x2="53.2" y2="80.29" width="2" layer="16"/>
 <wire x1="53.2" y1="80.29" x2="53.2" y2="79.7" width="2" layer="16"/>
-<wire x1="37.6" y1="18.7" x2="45.1" y2="11.2" width="2" layer="16"/>
+<wire x1="37.6" y1="18.7" x2="42.63" y2="13.67" width="2" layer="16"/>
+<wire x1="42.63" y1="13.67" x2="43.1" y2="13.2" width="2" layer="16"/>
 <wire x1="37.6" y1="18.7" x2="37.51" y2="18.7" width="2" layer="1"/>
 <wire x1="37.51" y1="18.7" x2="31.48" y2="24.73" width="2" layer="1"/>
@@
 <wire x1="94.835" y1="18.775" x2="103.61" y2="10" width="2" layer="1"/>
 <wire x1="76" y1="29.6" x2="89.2" y2="29.6" width="2" layer="1"/>
-<wire x1="71.6" y1="34" x2="76" y2="29.6" width="2" layer="16"/>
+<wire x1="72.13" y1="33.47" x2="76" y2="29.6" width="2" layer="16"/>
 <wire x1="71.8" y1="22.7" x2="71.75" y2="22.75" width="2" layer="16"/>
 <wire x1="76" y1="65.4" x2="76" y2="65" width="2" layer="16"/>
@@
 <wire x1="76.35" y1="2.12" x2="74.72" y2="3.75" width="2" layer="16"/>
 <contactref element="K83" pad="P$1"/>
-<wire x1="71.6" y1="34" x2="60.09" y2="34" width="2" layer="16"/>
-<wire x1="60.09" y1="34" x2="57.44" y2="36.65" width="2" layer="16"/>
-<wire x1="57.44" y1="36.65" x2="57.44" y2="39.98" width="2" layer="16"/>
-<wire x1="61.46" y1="44" x2="66.5" y2="44" width="2" layer="16"/>
-<wire x1="57.44" y1="39.98" x2="61.46" y2="44" width="2" layer="16"/>
+<wire x1="72.13" y1="33.47" x2="59.68" y2="33.47" width="2" layer="16"/>
+<wire x1="59.68" y1="33.47" x2="57.44" y2="35.71" width="2" layer="16"/>
+<wire x1="57.44" y1="35.71" x2="57.44" y2="40.77" width="2" layer="16"/>
+<wire x1="60.67" y1="44" x2="66.5" y2="44" width="2" layer="16"/>
+<wire x1="57.44" y1="40.77" x2="60.67" y2="44" width="2" layer="16"/>
 <wire x1="14.75" y1="41.75" x2="14.75" y2="45.25" width="2" layer="16"/>
 <wire x1="14.75" y1="45.25" x2="12" y2="48" width="2" layer="16"/>
@@
 <wire x1="109.8" y1="41.8" x2="109.75" y2="41.75" width="2" layer="16"/>
 <wire x1="109.8" y1="60.7" x2="109.75" y2="60.75" width="2" layer="16"/>
-<wire x1="20.6" y1="9.6" x2="14.75" y2="3.75" width="2" layer="16"/>
-<wire x1="20.6" y1="9.7" x2="20.6" y2="9.6" width="2" layer="16"/>
-<wire x1="24.44" y1="13.54" x2="20.6" y2="9.7" width="2" layer="16"/>
+<wire x1="24.44" y1="13.54" x2="21.72" y2="10.82" width="2" layer="16"/>
 <wire x1="35.86" y1="13.54" x2="24.44" y2="13.54" width="2" layer="16"/>
 <wire x1="90.87" y1="8" x2="94.31" y2="4.56" width="2" layer="1"/>
@@
 <wire x1="128" y1="48.8" x2="133.14" y2="53.94" width="2" layer="1"/>
 <wire x1="133.14" y1="53.94" x2="133.14" y2="66.53" width="2" layer="1"/>
+<wire x1="14.75" y1="3.75" x2="14.75" y2="8.75" width="2" layer="16"/>
+<wire x1="16.82" y1="10.82" x2="21.72" y2="10.82" width="2" layer="16"/>
+<wire x1="14.75" y1="8.75" x2="16.82" y2="10.82" width="2" layer="16"/>
 </signal>
 <signal name="COL6">
@@
 <via x="200.2" y="9.8" extent="1-16" drill="2"/>
 <via x="256.92" y="14.5" extent="1-16" drill="2"/>
-<wire x1="27.3" y1="7.9" x2="23" y2="7.9" width="2" layer="16"/>
-<wire x1="29.3" y1="9.9" x2="27.3" y2="7.9" width="2" layer="16"/>
+<wire x1="24.21" y1="7.9" x2="23" y2="7.9" width="2" layer="16"/>
+<wire x1="29.3" y1="9.9" x2="26.21" y2="9.9" width="2" layer="16"/>
+<wire x1="26.21" y1="9.9" x2="24.21" y2="7.9" width="2" layer="16"/>
 <wire x1="29.7" y1="9.5" x2="29.3" y2="9.9" width="2" layer="1"/>
 <wire x1="55.9" y1="9.5" x2="29.7" y2="9.5" width="2" layer="1"/>
@@
 <wire x1="99" y1="27.4" x2="99" y2="27.3495" width="2" layer="16"/>
 <wire x1="80.9" y1="27.4" x2="80" y2="27.3495" width="2" layer="16"/>
-<wire x1="15.1" y1="8.4" x2="4.5" y2="8.4" width="2" layer="16"/>
-<wire x1="22.8" y1="16.1" x2="15.1" y2="8.4" width="2" layer="16"/>
-<wire x1="29.31" y1="16.1" x2="22.8" y2="16.1" width="2" layer="16"/>
-<wire x1="41.9" y1="26.9" x2="39.545" y2="24.545" width="2" layer="16"/>
+<wire x1="20.35" y1="13.65" x2="22.8" y2="16.1" width="2" layer="16"/>
+<wire x1="22.8" y1="16.1" x2="29.31" y2="16.1" width="2" layer="16"/>
+<wire x1="40.11" y1="26.9" x2="38.65" y2="25.44" width="2" layer="16"/>
 <wire x1="38.65" y1="25.44" x2="29.31" y2="16.1" width="2" layer="16"/>
-<wire x1="42.2" y1="26.9" x2="41.9" y2="26.9" width="2" layer="16"/>
-<wire x1="4.5" y1="8.4" x2="4.5" y2="8.3495" width="2" layer="16"/>
+<wire x1="42.2" y1="26.9" x2="40.11" y2="26.9" width="2" layer="16"/>
 <wire x1="42.2" y1="26.9" x2="42.25" y2="26.9745" width="2" layer="16"/>
 <wire x1="6.9" y1="98.3" x2="19.1" y2="98.3" width="2" layer="1"/>
@@
 <wire x1="38.01" y1="42.73" x2="38.01" y2="28.4" width="2" layer="1"/>
 <wire x1="36.85" y1="27.24" x2="38.01" y2="28.4" width="2" layer="1"/>
-<wire x1="39.545" y1="24.545" x2="38.65" y2="25.44" width="2" layer="16"/>
 <wire x1="38.65" y1="25.44" x2="36.85" y2="27.24" width="2" layer="16"/>
 <wire x1="19.1" y1="98.3" x2="19.115" y2="98.315" width="2" layer="1"/>
-<wire x1="57.9" y1="26.9" x2="60.1" y2="26.9" width="2" layer="16"/>
-<wire x1="57.8" y1="26.8" x2="57.9" y2="26.9" width="2" layer="16"/>
-<wire x1="48.9" y1="26.8" x2="57.8" y2="26.8" width="2" layer="16"/>
-<wire x1="48.4" y1="27.3" x2="48.9" y2="26.8" width="2" layer="16"/>
-<wire x1="43.2" y1="27.3" x2="48.4" y2="27.3" width="2" layer="16"/>
-<wire x1="60.1" y1="26.9" x2="61" y2="27.3495" width="2" layer="16"/>
-<wire x1="43.2" y1="27.3" x2="42.25" y2="26.9745" width="2" layer="16"/>
+<wire x1="58.17475" y1="30.17475" x2="61" y2="27.3495" width="2" layer="16"/>
+<wire x1="42.5713375" y1="27.2958375" x2="42.25" y2="26.9745" width="2" layer="16"/>
 <wire x1="180.6" y1="45.8" x2="180.6" y2="29" width="2" layer="1"/>
 <wire x1="172.7" y1="45.8" x2="180.6" y2="45.8" width="2" layer="1"/>
@@
 <wire x1="33.27" y1="63.81" x2="32.2587875" y2="63.8176625" width="2" layer="1"/>
 <wire x1="32.2587875" y1="63.8176625" x2="30.434340625" y2="60.63" width="2" layer="1"/>
+<wire x1="10.7205" y1="13.65" x2="5.42" y2="8.3495" width="2" layer="16"/>
+<wire x1="4.5" y1="8.3495" x2="5.42" y2="8.3495" width="2" layer="16"/>
+<wire x1="10.7205" y1="13.65" x2="20.35" y2="13.65" width="2" layer="16"/>
+<wire x1="58.17475" y1="30.17475" x2="45.47475" y2="30.17475" width="2" layer="16"/>
+<wire x1="45.47475" y1="30.17475" x2="42.2" y2="26.9" width="2" layer="16"/>
 <wire x1="132.11" y1="87.52" x2="162" y2="88" width="0" layer="19" extent="1-1"/>
 </signal>
