File: atmega embedded main - za drugog Marka.sch (EAGLE design)
At the start: 150 parts, among them IC1 ATMEGA328PROUND, K100 SWITCH, K101 SWITCH, K102 SWITCH, K103 SWITCH, K104 SWITCH, K105 SWITCH, K106 SWITCH, K107 SWITCH, K108 SWITCH, K109 SWITCH, K110 SWITCH, K111 SWITCH, K112 SWITCH, K113 SWITCH, K114 SWITCH, K115 SWITCH, K116 SWITCH, K117 SWITCH, K118 SWITCH, K119 SWITCH, K120 SWITCH, K121 SWITCH, K122 SWITCH, K123 SWITCH, K124 SWITCH, K125 SWITCH, K126 SWITCH, K127 SWITCH, K128 SWITCH, K129 SWITCH, K130 SWITCH, K60 SWITCH, K67 SWITCH, K68 SWITCH, K69 SWITCH, K70 SWITCH, K71 SWITCH, K72 SWITCH, K73 SWITCH, K74 SWITCH, K75 SWITCH, K76 SWITCH, K77 SWITCH, K78 SWITCH, K79 SWITCH, K80 SWITCH, K81 SWITCH, K82 SWITCH, K83 SWITCH, K84 SWITCH, K85 SWITCH, K86 SWITCH, K87 SWITCH, K88 SWITCH, K89 SWITCH, K90 SWITCH, K91 SWITCH, K92 SWITCH, K93 SWITCH, K94 SWITCH, K95 SWITCH, K96 SWITCH, K97 SWITCH, K98 SWITCH, K99 SWITCH

Commit message: Finalized logic and started work on Marko's layout
Parts:
- removed D129, D130: (no value), adafruit:DIODESMA
- removed K129, K130: SWITCH, keyboard_switch:SWITCH
- added D3, D4, D5: (no value), adafruit:DIODESMA
- added K1, K2, K3: SWITCH, keyboard_switch:SWITCH
Connections:
- new net N$71: D3.C, K1.P$1
- net COL10: now also K3.P$2
- net COL2: now also K1.P$2
- net COL5: no longer K130.P$2
- net COL6: now also K128.P$2; no longer K129.P$2
- net COL7: now also K123.P$2; no longer K128.P$2
- net COL8: now also K117.P$2; no longer K123.P$2
- net COL9: now also K2.P$2; no longer K117.P$2
- net N$26: now also D5.C, K3.P$1; no longer D129.C, K129.P$1
- net N$35: now also D4.C, K2.P$1; no longer D130.C, K130.P$1
- net ROW4: now also D3.A, D5.A, IC1.(PCI1/OC1A/OC1S)PB1; no longer IC1.(PCI2/SS/OC1B)PB2
- net ROW5: now also IC1.(PCI3/MOSI/OC2A)PB3; no longer D129.A, D130.A, IC1.(PCI1/OC1A/OC1S)PB1
- net ROW6: now also D4.A, IC1.(PCI2/SS/OC1B)PB2; no longer IC1.(PCI3/MOSI/OC2A)PB3
Other:
- moved on the sheet: D111, D125, D128, D86, D87, D97, D98, K117, K118, K122, K124, K88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

Commit message: Wired up connectors
Connections:
- net N$15 renamed RESET
Changed lines of the file:
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@@
 </segment>
 </net>
-<net name="N$15" class="0">
+<net name="RESET" class="0">
 <segment>
 <pinref part="R5" gate="G$1" pin="2"/>

Commit message: Test 1
Connections:
- net COL1: now also K87.P$2; no longer K94.P$2
- net COL2: now also K94.P$2; no longer K95.P$2
- net COL3: now also K95.P$2; no longer K96.P$2
- net COL4: now also K96.P$2; no longer K87.P$2, K97.P$2
- net ROW4: now also D81.A; no longer D87.A
- net ROW5: now also D87.A; no longer D86.A
- net ROW6: no longer D81.A
- net ROW7: now also D86.A
Other:
- moved on the sheet: D81, D83, D84, D85, D86, D87, D97, K87, K88, K92, K94, K95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

Commit message: Test2
Connections:
- removed net N$66: D127.C, K123.P$1
- new net N$15: D98.C, K118.P$2
- net COL1: now also D86.A
- net COL2: now also K72.P$1; no longer K72.P$2
- net COL6: now also K118.P$1, K119.P$1; no longer K118.P$2, K119.P$2
- net COL7: now also K123.P$1; no longer K123.P$2
- net N$36: now also K72.P$2; no longer K72.P$1
- net N$41: now also D119.C, K119.P$2; no longer D98.C, K118.P$1
- net N$43: now also D127.C, K123.P$2; no longer D119.C, K119.P$1
- net ROW4: now also D82.A; no longer D81.A
- net ROW6: now also D81.A; no longer D82.A
- net ROW7: now also K97.P$2; no longer D86.A
Other:
- moved on the sheet: D119, D127, D72, D81, D82, D86, D98, K118, K119, K87, K93

Commit message: Horrible design
Connections:
- net COL2: now also K82.P$1; no longer K82.P$2
- net COL3: now also K83.P$1; no longer K83.P$2
- net COL6: now also K118.P$2; no longer K118.P$1
- net N$11: now also K82.P$2; no longer K82.P$1
- net N$15: now also K118.P$1; no longer K118.P$2
- net N$22: now also K83.P$2; no longer K83.P$1
Other:
- moved on the sheet: D89, D91, K82, K83, K93
